File: pcb/LLV1/LLV1.kicad_pcb (KiCad board)
At the start: 2 copper layers, 1 part

Commit message: Completed initial PCB schematic
Parts:
- removed REF**: Val**, Seeed_Studio_XIAO_Series:XIAO-nRF52840-SMD
- added J2: Conn_01x02, Connector_JST:JST_PH_S2B-PH-SM4-TB_1x02-1MP_P2.00mm_Horizontal, F.Cu at (136.0, 150.0)
- added U1: XIAO-nRF52840-SMD, Seeed_Studio_XIAO_Series:XIAO-nRF52840-SMD, F.Cu at (131.7, 144.6)
- added U2: MAX30102, OptoDevice:Maxim_OLGA-14_3.3x5.6mm_P0.8mm, F.Cu at (128.7, 136.6)
- added U3: ATGM336H-5N31, ATGM336H-5N31:GPSM-SMD_ATGM336H-TR, F.Cu at (172.5, 151.5)

Commit message: Updated PCB layout
Parts:
- removed U3: ATGM336H-5N31, ATGM336H-5N31:GPSM-SMD_ATGM336H-TR
- added SW1: SW_Push, easyeda2kicad:KEY-SMD_4P-L4.8-W4.6-P1.70-LS6.2, F.Cu at (140.3, 148.6)
- U2: footprint OptoDevice:Maxim_OLGA-14_3.3x5.6mm_P0.8mm -> MAX30102_BREAKOUT:Untitled; moved to B.Cu
- moved J2 26.9 mm to (156.6, 132.7), turned to -90 degrees
- moved U2 5.60 mm to (133.3, 139.7), turned to -90 degrees
Connections:
- U1 pad 1: unconnected-(U1-D0-Pad1) -> Net-(U1-D0)
- U1 pad 8: Net-(U1-D7) -> unconnected-(U1-D7-Pad8)
- U1 pad 9: Net-(U1-D8) -> unconnected-(U1-D8-Pad9)

Commit message: Sync repo with latest code
Parts:
- J2: footprint Connector_JST:JST_PH_S2B-PH-SM4-TB_1x02-1MP_P2.00mm_Horizontal -> Connector_JST:JST_PH_S2B-PH-K_1x02_P2.00mm_Horizontal
- moved J2 20.0 mm to (145.9, 149.7), turned to 90 degrees
- moved SW1 2.66 mm to (138.4, 150.4)
- moved U2 1.81 mm to (132.8, 138.0)
Routing:
- net GND: track 0.00 -> 61.3 mm
- net +3V3: track 0.00 -> 38.0 mm
- net Net-(U1-D0): track 0.00 -> 27.3 mm
- net Net-(J2-Pin_1): track 0.00 -> 19.9 mm
- net Net-(U1-D5): track 0.00 -> 4.83 mm
- net Net-(U1-D4): track 0.00 -> 4.83 mm
Other:
- board outline added: 28.8 x 30.3 mm

Commit message: Updated PCB layout
Parts:
- moved SW1 3.88 mm to (134.5, 150.4)
Routing:
- net +3V3: track 38.0 -> 22.1 mm, vias 0 -> 1
- net GND: track 61.3 -> 46.5 mm
- net Net-(U1-D0): track 27.3 -> 25.7 mm
- net Net-(J2-Pin_1): track 19.9 -> 21.2 mm
Changed lines of the file:
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@@
 	(footprint "easyeda2kicad:KEY-SMD_4P-L4.8-W4.6-P1.70-LS6.2"
 		(layer "F.Cu")
-		(at 138.3792 150.368)
+		(at 134.5 150.368)
 		(property "Reference" "SW1"
 			(at 0 -3.205 0)
@@
 	)
 	(segment
-		(start 145.419 139.902)
-		(end 145.419 147.1716)
-		(width 0.3)
-		(layer "F.Cu")
-		(net "GND")
-	)
-	(segment
-		(start 147.1226 148.8752)
-		(end 145.8976 147.6502)
-		(width 0.3)
-		(layer "F.Cu")
-		(net "GND")
-	)
-	(segment
-		(start 146.778056 150.6002)
-		(end 147.1226 150.255656)
-		(width 0.3)
-		(layer "F.Cu")
-		(net "GND")
-	)
-	(segment
-		(start 135.7792 149.518)
-		(end 136.6292 150.368)
+		(start 127.7366 141.7828)
+		(end 131.9 145.9462)
 		(width 0.3)
 		(layer "F.Cu")
@@
 	)
 	(segment
-		(start 136.6292 150.368)
-		(end 144.784944 150.368)
-		(width 0.3)
-		(layer "F.Cu")
-		(net "GND")
-	)
-	(segment
 		(start 138.064 131.892)
 		(end 141.874 128.082)
@@
 	)
 	(segment
+		(start 138.392 131.892)
+		(end 142.5 136)
+		(width 1)
+		(layer "F.Cu")
+		(net "GND")
+	)
+	(segment
 		(start 142.8225 129.0305)
 		(end 148.714 129.0305)
@@
 	)
 	(segment
-		(start 127.7366 141.7828)
-		(end 135.4718 149.518)
-		(width 0.3)
-		(layer "F.Cu")
-		(net "GND")
-	)
-	(segment
-		(start 137.409 131.892)
-		(end 145.419 139.902)
-		(width 0.3)
-		(layer "F.Cu")
-		(net "GND")
-	)
-	(segment
-		(start 135.4718 149.518)
-		(end 135.7792 149.518)
-		(width 0.3)
-		(layer "F.Cu")
-		(net "GND")
-	)
-	(segment
-		(start 145.017144 150.6002)
-		(end 146.778056 150.6002)
-		(width 0.3)
-		(layer "F.Cu")
-		(net "GND")
-	)
-	(segment
-		(start 136.159 131.892)
-		(end 137.409 131.892)
-		(width 0.3)
-		(layer "F.Cu")
-		(net "GND")
-	)
-	(segment
 		(start 136.159 131.892)
 		(end 138.064 131.892)
@@
 	)
 	(segment
-		(start 144.784944 150.368)
-		(end 145.017144 150.6002)
-		(width 0.3)
+		(start 136.159 131.892)
+		(end 138.392 131.892)
+		(width 1)
 		(layer "F.Cu")
 		(net "GND")
 	)
 	(segment
-		(start 147.1226 150.255656)
-		(end 147.1226 148.8752)
-		(width 0.3)
+		(start 144.6502 147.6502)
+		(end 145.8976 147.6502)
+		(width 1)
 		(layer "F.Cu")
 		(net "GND")
 	)
 	(segment
-		(start 140.9792 149.518)
-		(end 134.274 142.8128)
+		(start 131.9 145.9462)
+		(end 131.9 149.518)
+		(width 0.3)
+		(layer "F.Cu")
+		(net "GND")
+	)
+	(segment
+		(start 142.5 136)
+		(end 142.5 145.5)
+		(width 1)
+		(layer "F.Cu")
+		(net "GND")
+	)
+	(segment
+		(start 142.5 145.5)
+		(end 144.6502 147.6502)
+		(width 1)
+		(layer "F.Cu")
+		(net "GND")
+	)
+	(segment
+		(start 134.5 144.5)
+		(end 134.5 127.0665)
+		(width 0.3)
+		(layer "F.Cu")
+		(net "Net-(U1-D0)")
+	)
+	(segment
+		(start 137.1 149.518)
+		(end 137.1 147.1)
 		(width 0.3)
 		(layer "F.Cu")
@@
 	)
 	(segment
-		(start 134.274 126.8405)
+		(start 134.5 127.0665)
 		(end 133.924 126.4905)
 		(width 0.3)
@@
 	)
 	(segment
-		(start 134.274 142.8128)
-		(end 134.274 126.8405)
+		(start 137.1 147.1)
+		(end 134.5 144.5)
 		(width 0.3)
 		(layer "F.Cu")
@@
 	)
 	(segment
-		(start 150.439 131.2205)
-		(end 150.439 125.631146)
+		(start 148.714 131.5705)
+		(end 140.5705 131.5705)
 		(width 0.3)
 		(layer "F.Cu")
@@
 	)
 	(segment
-		(start 127.7366 128.718546)
+		(start 140.5 131.5)
+		(end 140.5705 131.5705)
+		(width 0.3)
+		(layer "F.Cu")
+		(net "+3V3")
+	)
+	(via
+		(at 140.5 131.5)
+		(size 0.6)
+		(drill 0.3)
+		(layers "F.Cu" "B.Cu")
+		(net "+3V3")
+	)
+	(segment
+		(start 137.8372 134.1628)
 		(end 127.7366 134.1628)
 		(width 0.3)
-		(layer "F.Cu")
+		(layer "B.Cu")
 		(net "+3V3")
 	)
 	(segment
-		(start 150.439 125.631146)
-		(end 149.149854 124.342)
-		(width 0.3)
-		(layer "F.Cu")
+		(start 140.5 131.5)
+		(end 137.8372 134.1628)
+		(width 0.3)
+		(layer "B.Cu")
 		(net "+3V3")
 	)
 	(segment
-		(start 149.149854 124.342)
-		(end 132.113146 124.342)
-		(width 0.3)
-		(layer "F.Cu")
-		(net "+3V3")
-	)
-	(segment
-		(start 132.113146 124.342)
-		(end 127.7366 128.718546)
-		(width 0.3)
-		(layer "F.Cu")
-		(net "+3V3")
-	)
-	(segment
-		(start 148.714 131.5705)
-		(end 150.089 131.5705)
-		(width 0.3)
-		(layer "F.Cu")
-		(net "+3V3")
-	)
-	(segment
-		(start 150.089 131.5705)
-		(end 150.439 131.2205)
-		(width 0.3)
-		(layer "F.Cu")
-		(net "+3V3")
-	)
-	(segment
-		(start 136.159 139.9116)
+		(start 140 146)
+		(end 143.6502 149.6502)
+		(width 1)
+		(layer "F.Cu")
+		(net "Net-(J2-Pin_1)")
+	)
+	(segment
+		(start 143.6502 149.6502)
 		(end 145.8976 149.6502)
-		(width 0.3)
+		(width 1)
 		(layer "F.Cu")
 		(net "Net-(J2-Pin_1)")
@@
 	(segment
 		(start 136.159 133.797)
-		(end 136.159 139.9116)
-		(width 0.3)
+		(end 140 137.638)
+		(width 1)
 		(layer "F.Cu")
 		(net "Net-(J2-Pin_1)")
+	)
+	(segment
+		(start 140 137.638)
+		(end 140 146)
+		(width 1)
+		(layer "F.Cu")
+		(net "Net-(J2-Pin_1)")
