File: pcb/LLV1/LLV1.kicad_sch (KiCad schematic)
At the start: 4 parts, among them J2 Conn_01x02, U1 XIAO-nRF52840-SMD, U2 MAX30102, U3 ATGM336H-5N31

Commit message: Updated PCB schematic
Connections:
- net +3V3: now also U3.8 (VCC)
- net GND: now also U3.1 (GND)
- net at U3.2 (TXD): now also U1.8 (D7)
- net at U3.3 (RXD): now also U1.9 (D8)
Changed lines of the file:
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@@
+	(wire
+		(pts
+			(xy 172.72 102.87) (xy 187.96 102.87)
+		)
+		(stroke
+			(width 0)
+			(type default)
+		)
+	)
 	(wire
 		(pts
@@
 	(wire
 		(pts
+			(xy 182.88 97.79) (xy 187.96 97.79)
+		)
+		(stroke
+			(width 0)
+			(type default)
+		)
+	)
+	(wire
+		(pts
+			(xy 171.45 114.3) (xy 171.45 100.33)
+		)
+		(stroke
+			(width 0)
+			(type default)
+		)
+	)
+	(wire
+		(pts
 			(xy 71.12 130.81) (xy 71.12 110.49)
 		)
@@
 	(wire
 		(pts
+			(xy 171.45 100.33) (xy 187.96 100.33)
+		)
+		(stroke
+			(width 0)
+			(type default)
+		)
+	)
+	(wire
+		(pts
 			(xy 125.73 138.43) (xy 125.73 120.65)
 		)
@@
 	(wire
 		(pts
+			(xy 182.88 115.57) (xy 187.96 115.57)
+		)
+		(stroke
+			(width 0)
+			(type default)
+		)
+	)
+	(wire
+		(pts
 			(xy 96.52 146.05) (xy 96.52 148.59)
 		)
@@
 	(wire
 		(pts
+			(xy 149.86 110.49) (xy 172.72 110.49)
+		)
+		(stroke
+			(width 0)
+			(type default)
+		)
+	)
+	(wire
+		(pts
 			(xy 88.9 118.11) (xy 88.9 120.65)
 		)
@@
 	(wire
 		(pts
+			(xy 172.72 110.49) (xy 172.72 102.87)
+		)
+		(stroke
+			(width 0)
+			(type default)
+		)
+	)
+	(wire
+		(pts
 			(xy 134.62 138.43) (xy 125.73 138.43)
 		)
@@
 		(pts
 			(xy 149.86 99.06) (xy 161.29 99.06)
+		)
+		(stroke
+			(width 0)
+			(type default)
+		)
+	)
+	(wire
+		(pts
+			(xy 149.86 114.3) (xy 171.45 114.3)
 		)
 		(stroke
@@
 					(unit 1)
 				)
+			)
+		)
+	)
+	(symbol
+		(lib_id "power:+3V3")
+		(at 182.88 115.57 90)
+		(unit 1)
+		(body_style 1)
+		(exclude_from_sim no)
+		(in_bom yes)
+		(on_board yes)
+		(in_pos_files yes)
+		(dnp no)
+		(fields_autoplaced yes)
+		(property "Reference" "#PWR09"
+			(at 186.69 115.57 0)
+			(hide yes)
+			(show_name no)
+			(do_not_autoplace no)
+			(effects
+				(font
+					(size 1.27 1.27)
+				)
+			)
+		)
+		(property "Value" "+3V3"
+			(at 179.07 115.5699 90)
+			(show_name no)
+			(do_not_autoplace no)
+			(effects
+				(font
+					(size 1.27 1.27)
+				)
+				(justify left)
+			)
+		)
+		(property "Footprint" ""
+			(at 182.88 115.57 0)
+			(hide yes)
+			(show_name no)
+			(do_not_autoplace no)
+			(effects
+				(font
+					(size 1.27 1.27)
+				)
+			)
+		)
+		(property "Datasheet" ""
+			(at 182.88 115.57 0)
+			(hide yes)
+			(show_name no)
+			(do_not_autoplace no)
+			(effects
+				(font
+					(size 1.27 1.27)
+				)
+			)
+		)
+		(property "Description" "Power symbol creates a global label with name \"+3V3\""
+			(at 182.88 115.57 0)
+			(hide yes)
+			(show_name no)
+			(do_not_autoplace no)
+			(effects
+				(font
+					(size 1.27 1.27)
+				)
+			)
+		)
+		(pin "1"
+		)
+		(instances
+			(project "LLV1"
+				(path "/b501725e-37bd-468e-b174-d4f4e10a500b"
+					(reference "#PWR09")
+					(unit 1)
+				)
+			)
+		)
+	)
+	(symbol
+		(lib_id "power:GND")
+		(at 182.88 97.79 270)
+		(unit 1)
+		(body_style 1)
+		(exclude_from_sim no)
+		(in_bom yes)
+		(on_board yes)
+		(in_pos_files yes)
+		(dnp no)
+		(fields_autoplaced yes)
+		(property "Reference" "#PWR08"
+			(at 176.53 97.79 0)
+			(hide yes)
+			(show_name no)
+			(do_not_autoplace no)
+			(effects
+				(font
+					(size 1.27 1.27)
+				)
+			)
+		)
+		(property "Value" "GND"
+			(at 179.07 97.7899 90)
+			(show_name no)
+			(do_not_autoplace no)
+			(effects
+				(font
+					(size 1.27 1.27)
+				)
+				(justify right)
+			)
+		)
+		(property "Footprint" ""
+			(at 182.88 97.79 0)
+			(hide yes)
+			(show_name no)
+			(do_not_autoplace no)
+			(effects
+				(font
+					(size 1.27 1.27)
+				)
+			)
+		)
+		(property "Datasheet" ""
+			(at 182.88 97.79 0)
+			(hide yes)
+			(show_name no)
+			(do_not_autoplace no)
+			(effects
+				(font
+					(size 1.27 1.27)
+				)
+			)
+		)
+		(property "Description" "Power symbol creates a global label with name \"GND\" , ground"
+			(at 182.88 97.79 0)
+			(hide yes)
+			(show_name no)
+			(do_not_autoplace no)
+			(effects
+				(font
+					(size 1.27 1.27)
+				)
+			)
+		)
+		(pin "1"
+		)
+		(instances
+			(project "LLV1"
+				(path "/b501725e-37bd-468e-b174-d4f4e10a500b"
+					(reference "#PWR08")
+					(unit 1)
+				)

Commit message: Completed initial PCB schematic
Parts:
- U3: footprint easyeda2kicad:GPSM-SMD_ATGM336H-TR -> ATGM336H-5N31:GPSM-SMD_ATGM336H-TR
Changed lines of the file:
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@@
 			)
 		)
-		(property "Footprint" "easyeda2kicad:GPSM-SMD_ATGM336H-TR"
+		(property "Footprint" "ATGM336H-5N31:GPSM-SMD_ATGM336H-TR"
 			(at 204.47 125.73 0)
 			(hide yes)

Commit message: Updated PCB layout
Parts:
- removed U3: ATGM336H-5N31, ATGM336H-5N31:GPSM-SMD_ATGM336H-TR, symbol ATGM336H-5N31:ATGM336H-5N31
- added SW1: SW_Push, easyeda2kicad:KEY-SMD_4P-L4.8-W4.6-P1.70-LS6.2, symbol Switch:SW_Push
- U2: footprint OptoDevice:Maxim_OLGA-14_3.3x5.6mm_P0.8mm -> MAX30102_BREAKOUT:Untitled
Connections:
- net GND: now also SW1.1
- net at U1.1 (D0): now also SW1.2

Commit message: Sync repo with latest code
Parts:
- J2: footprint (none) -> Connector_JST:JST_PH_S2B-PH-K_1x02_P2.00mm_Horizontal
Changed lines of the file:
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@@
 			)
 		)
-		(property "Footprint" ""
+		(property "Footprint" "Connector_JST:JST_PH_S2B-PH-K_1x02_P2.00mm_Horizontal"
 			(at 139.7 138.43 0)
 			(hide yes)

Commit message: Update PCB layout
Parts:
- J2: footprint Connector_JST:JST_PH_S2B-PH-K_1x02_P2.00mm_Horizontal -> Materials:JST_S2B-PH-SM4-TB
Changed lines of the file:
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@@
 			)
 		)
-		(property "Footprint" "Connector_JST:JST_PH_S2B-PH-K_1x02_P2.00mm_Horizontal"
+		(property "Footprint" "Materials:JST_S2B-PH-SM4-TB"
 			(at 139.7 138.43 0)
 			(hide yes)

Commit message: Initial PCB complete & fall detection improvments
Connections:
- net at SW1.2: now also U1.4 (D3); no longer U1.1 (D0)
Other:
- moved on the sheet: SW1
Changed lines of the file:
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@@
 	(generator_version "10.0")
 	(paper "A4")
-	(junction
-		(at 111.76 91.44)
-		(diameter 0)
-		(color 0 0 0 0)
-	)
 	(wire
 		(pts
@@
 	(wire
 		(pts
-			(xy 96.52 91.44) (xy 111.76 91.44)
-		)
-		(stroke
-			(width 0)
-			(type default)
-		)
-	)
-	(wire
-		(pts
-			(xy 111.76 91.44) (xy 113.03 91.44)
-		)
-		(stroke
-			(width 0)
-			(type default)
-		)
-	)
-	(wire
-		(pts
 			(xy 71.12 130.81) (xy 71.12 110.49)
 		)
@@
 	(wire
 		(pts
-			(xy 80.01 91.44) (xy 86.36 91.44)
+			(xy 83.82 102.87) (xy 86.36 102.87)
 		)
 		(stroke
@@
 		(pts
 			(xy 149.86 99.06) (xy 161.29 99.06)
+		)
+		(stroke
+			(width 0)
+			(type default)
+		)
+	)
+	(wire
+		(pts
+			(xy 111.76 102.87) (xy 96.52 102.87)
 		)
 		(stroke
@@
 	(symbol
 		(lib_id "Switch:SW_Push")
-		(at 91.44 91.44 0)
+		(at 91.44 102.87 0)
 		(unit 1)
 		(body_style 1)
@@
 		(fields_autoplaced yes)
 		(property "Reference" "SW1"
-			(at 91.44 83.82 0)
+			(at 91.44 95.25 0)
 			(show_name no)
 			(do_not_autoplace no)
@@
 		)
 		(property "Value" "SW_Push"
-			(at 91.44 86.36 0)
+			(at 91.44 97.79 0)
 			(show_name no)
 			(do_not_autoplace no)
@@
 		)
 		(property "Footprint" "easyeda2kicad:KEY-SMD_4P-L4.8-W4.6-P1.70-LS6.2"
-			(at 91.44 86.36 0)
+			(at 91.44 97.79 0)
 			(hide yes)
 			(show_name no)
@@
 		)
 		(property "Datasheet" ""
-			(at 91.44 86.36 0)
+			(at 91.44 97.79 0)
 			(hide yes)
 			(show_name no)
@@
 		)
 		(property "Description" "Push button switch, generic, two pins"
-			(at 91.44 91.44 0)
+			(at 91.44 102.87 0)
 			(hide yes)
 			(show_name no)
@@
 	(symbol
 		(lib_id "power:GND")
-		(at 80.01 91.44 270)
+		(at 83.82 102.87 270)
 		(unit 1)
 		(body_style 1)
@@
 		(fields_autoplaced yes)
 		(property "Reference" "#PWR08"
-			(at 73.66 91.44 0)
+			(at 77.47 102.87 0)
 			(hide yes)
 			(show_name no)
@@
 		)
 		(property "Value" "GND"
-			(at 76.2 91.4399 90)
+			(at 80.01 102.8699 90)
 			(show_name no)
 			(do_not_autoplace no)
@@
 		)
 		(property "Footprint" ""
-			(at 80.01 91.44 0)
+			(at 83.82 102.87 0)
 			(hide yes)
 			(show_name no)
@@
 		)
 		(property "Datasheet" ""
-			(at 80.01 91.44 0)
+			(at 83.82 102.87 0)
 			(hide yes)
 			(show_name no)
@@
 		)
 		(property "Description" "Power symbol creates a global label with name \"GND\" , ground"
-			(at 80.01 91.44 0)
-			(hide yes)
-			(show_name no)
+			(at 83.82 102.87 0)
+			(hide yes)
+			(show_name no)
